Commit message: Initial attempt at robot state publisher.

File: src/pff/urdf/pff.urdf (robot description, URDF)
Before this commit: robot pff, 3 links, 2 joints
Joints:
- joint axle_to_left_wheel: origin xyz=0 0 0.4 -> xyz=0 0.4 0 rpy=1.57075 0 0
- joint axle_to_right_wheel: axis 0 1 0 -> 0 0 1; origin xyz=0 0 -0.4 -> xyz=0 -0.4 0 rpy=1.57075 0 0
